File: hardware/ae-tracker-db/ae-tracker-db.kicad_pcb (KiCad board)
At the start: 2 copper layers, 29 x 41.1 mm, 29 parts, among them J2 Conn_01x01_Pin, J3 Conn_01x04_Socket, J4 Conn_01x16_Pin, U1 SN65HVD231, U2 LIS3DH, U3 BQ25176J, U4 TPS1H000-Q1

Commit message: v0.0.2 WIP
Parts:
- F1: value Fuse_Small -> 1.5A 1206
Routing:
- net GND: track 29.5 -> 27.7 mm, vias 27 -> 26
- net Net-(U3-ISET): track 3.86 -> 5.17 mm

Commit message: Fixing wrong part number
Other:
- board text added: "JLCJLCJLCJLC"
- board text removed: "JLCJLCJLC"
Changed lines of the file:
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@@
 		(sheetname "/")
 		(sheetfile "ae-tracker-db.kicad_sch")
-		(attr through_hole exclude_from_pos_files exclude_from_bom dnp)
+		(attr through_hole exclude_from_pos_files dnp)
 		(fp_line
 			(start -1.38 -1.38)
@@
 			)
 		)
-		(property "LCSC" "C5370355"
+		(property "LCSC" "C2894958"
 			(at 0 0 180)
 			(unlocked yes)
@@
 		(sheetfile "ae-tracker-db.kicad_sch")
 		(zone_connect 1)
-		(attr exclude_from_pos_files exclude_from_bom allow_soldermask_bridges)
+		(attr exclude_from_pos_files allow_soldermask_bridges)
 		(net_tie_pad_groups "1, 2")
 		(fp_poly
@@
 		)
 	)
-	(gr_text "JLCJLCJLC"
+	(gr_text "JLCJLCJLCJLC"
 		(at 156.4 85.8 0)
 		(layer "B.SilkS")
